File: simlinkModule.kicad_sch (KiCad schematic)
At the start: 0 parts

Commit message: main pcb basic setup
Parts:
- added C? (x4): 0.1uF/50V(10%), symbol Device:C
- added C? (x3): 22uF/10V(20%), symbol Device:C
- added D?: RED LED, symbol Device:LED
- added J? (x2): Conn_01x06_Male, symbol Connector:Conn_01x06_Male
- added J?: Conn_01x08_Female, symbol Connector:Conn_01x08_Female
- added Q? (x2): Q_NPN_BEC, symbol Device:Q_NPN_BEC
- added R? (x3): 10K, symbol Device:R
- added R?: R, symbol Device:R
- added SW? (x2): SW_Push, symbol Switch:SW_Push
- added U?: ESP32-WROOM-E, Espressif:ESP32-WROOM-32E, symbol Espressif:ESP32-WROOM-E
- added U?: AMS1117-3.3, Package_TO_SOT_SMD:SOT-223-3_TabPin2, symbol Regulator_Linear:AMS1117-3.3
Connections:
- new net: Q?.1 (B), R?.2 (x2)
- new net: D?.2 (A), R?.2
- new net +3.3V: C?.1, C?.1, C?.1, J?.1 (Pin_1), R?.1, R?.1, U?.2 (3V3), U?.2 (VO)
- new net Boot: C?.2, Q?.2 (E), SW?.2, U?.25 (GPIO0/BOOT/ADC2_CH1)
- new net Btn_L: J?.5 (Pin_5), U?.11 (DAC_2/ADC2_CH9/GPIO26)
- new net Btn_R: J?.6 (Pin_6), U?.10 (DAC_1/ADC2_CH8/GPIO25)
- new net C-Data: J?.1 (Pin_1), U?.27 (GPIO16)
- new net CTS: J?.5 (Pin_5), Q?.2 (E), R?.1
- new net DTR: J?.6 (Pin_6), Q?.3 (C), R?.1
- new net EN: C?.1, C?.2, Q?.3 (C), R?.2, SW?.2, U?.3 (EN/CHIP_PU)
- new net GND: C?.1, C?.1, C?.2, C?.2, C?.2, C?.2, C?.2, D?.1 (K), J?.2 (Pin_2), J?.2 (Pin_2), J?.2 (Pin_2), SW?.1, SW?.1, U?.1 (GND), U?.1 (GND), U?.15 (GND), U?.38 (GND), U?.39 (GND_THERMAL)
- new net PR_RX: J?.4 (Pin_4), U?.34 (U0RXD/GPIO3)
- new net PR_TX: J?.3 (Pin_3), U?.35 (U0TXD/GPIO1)
- new net SCK: J?.4 (Pin_4), U?.36 (GPIO22)
- new net SDA: J?.3 (Pin_3), U?.33 (GPIO21)
- new net VCC: C?.1, J?.1 (Pin_1), J?.3 (Pin_3), U?.3 (VI)
- no-connect marks 0 -> 22
Other:
- added sheet IOBoard (ioboard.kicad_sch)
- note added: "Auto program for espflash DTR CTS --> EN Boot 1 1 1 1 0 0 1 1 1 0 0 1 0 1 1 0"
- note added: "Controller-Connector"
- note added: "ESP32 Module"
- note added: "Expansion-Port"
- note added: "Flash logic"
- note added: "Flash-Port"
- note added: "Power Supply"
- note added: "Switch Button"
- note added: "VCC = 3.3V / 5V"
- note added: "VCC = 6V"
- company: (none) -> Fabian Kuffer
- title: (none) -> Mainboard

Commit message: io board added
Parts:
- added J?: Conn_01x01, symbol Connector_Generic:Conn_01x01
- added R? (x2): 4.7K, symbol Device:R
Connections:
- net Boot: now also R?.2; no longer SW?.2
- net EN: now also R?.2; no longer SW?.2
- net ADC_OUT: now reaches U?.8 (32K_XP/GPIO32/ADC1_CH4)
- net ADC_OUT: now also J?.1 (Pin_1)
- new net: R?.1, SW?.2 (x2)
Other:
- note added: "internal pull-up: 45K"
- moved on the sheet: C?, SW?

Commit message: esc check done
Parts:
- added D2, D3: BAT760-7, symbol Diode:PMEG1020EH
- added D4: LESD8D3.3CAT5G, symbol Diode:1N62xxCA
- added D5: LESD8D12T5G, symbol Diode:PMEG1020EH
- C1, C2, C4: renamed from C?; value 22uF/10V(20%) -> 22u
- C3, C5, C6, C7: renamed from C?; value 0.1uF/50V(10%) -> 0.1u
- Q1, Q2: renamed from Q?; value Q_NPN_BEC -> SS8050-G
- R1: renamed from R?; value R -> 4.7K
- gave numbers to parts that had none: 14
Connections:
- net C-Data: now also D4.2 (A2)
- net GND: now also D4.1 (A1), D5.2 (A)
- net VCC: now also D2.1 (K), D2.2 (A), D3.1 (K), D3.2 (A), D5.1 (K)
Other:
- note added: "VCC = 6V..12V"
- note removed: "VCC = 6V"
- moved on the sheet: C1, C2, D1, J2, J3, J4, R1, U1
