File: ioBoard/ioBoard.kicad_pcb (KiCad board)
At the start: 2 copper layers, 35 x 41.9 mm, 23 parts, among them J1 Conn_01x06_Male, J2 Conn_01x14, SW1 C202424, SW2 C202424

Commit message: jlcpcb orders created
Changed lines of the file:
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@@
     (fp_line (start 1 0.625) (end -1 0.625) (layer "F.Fab") (width 0.1))
     (fp_line (start -1 -0.625) (end 1 -0.625) (layer "F.Fab") (width 0.1))
-    (pad "1" smd roundrect (at -1.0375 0) (size 1.175 1.45) (layers "F.Cu" "F.Paste" "F.Mask") (roundrect_rratio 0.212766)
+    (pad "1" smd roundrect (at -1.0375 0) (size 1.175 1.45) (layers "F.Cu" "F.Paste" "F.Mask") (roundrect_rratio 0.2127659574)
       (net 1 "Net-(C1-Pad1)") (pintype "passive"))
-    (pad "2" smd roundrect (at 1.0375 0) (size 1.175 1.45) (layers "F.Cu" "F.Paste" "F.Mask") (roundrect_rratio 0.212766)
+    (pad "2" smd roundrect (at 1.0375 0) (size 1.175 1.45) (layers "F.Cu" "F.Paste" "F.Mask") (roundrect_rratio 0.2127659574)
       (net 2 "Net-(C1-Pad2)") (pintype "passive"))
     (model "${KICAD6_3DMODEL_DIR}/Capacitor_SMD.3dshapes/C_0805_2012Metric.wrl"
@@
     (property "Sheetfile" "ioBoard.kicad_sch")
     (property "Sheetname" "")
-    (attr exclude_from_pos_files)
+    (attr exclude_from_pos_files exclude_from_bom)
     (fp_text reference "H4" (at 0 -3.2) (layer "F.Fab")
       (effects (font (size 1 1) (thickness 0.15)))
@@
     (fp_line (start -1 0.625) (end -1 -0.625) (layer "F.Fab") (width 0.1))
     (fp_line (start 1 -0.625) (end 1 0.625) (layer "F.Fab") (width 0.1))
-    (pad "1" smd roundrect (at -1.0375 0) (size 1.175 1.45) (layers "F.Cu" "F.Paste" "F.Mask") (roundrect_rratio 0.212766)
+    (pad "1" smd roundrect (at -1.0375 0) (size 1.175 1.45) (layers "F.Cu" "F.Paste" "F.Mask") (roundrect_rratio 0.2127659574)
       (net 3 "Net-(C2-Pad1)") (pintype "passive"))
-    (pad "2" smd roundrect (at 1.0375 0) (size 1.175 1.45) (layers "F.Cu" "F.Paste" "F.Mask") (roundrect_rratio 0.212766)
+    (pad "2" smd roundrect (at 1.0375 0) (size 1.175 1.45) (layers "F.Cu" "F.Paste" "F.Mask") (roundrect_rratio 0.2127659574)
       (net 4 "Net-(C2-Pad2)") (pintype "passive"))
     (model "${KICAD6_3DMODEL_DIR}/Capacitor_SMD.3dshapes/C_0805_2012Metric.wrl"
@@
     (property "Sheetfile" "ioBoard.kicad_sch")
     (property "Sheetname" "")
-    (attr exclude_from_pos_files)
+    (attr exclude_from_pos_files exclude_from_bom)
     (fp_text reference "H3" (at 0 -3.2) (layer "F.Fab")
       (effects (font (size 1 1) (thickness 0.15)))
@@
     (property "Sheetfile" "ioBoard.kicad_sch")
     (property "Sheetname" "")
-    (attr exclude_from_pos_files)
+    (attr exclude_from_pos_files exclude_from_bom)
     (fp_text reference "H2" (at 0 -3.2) (layer "F.Fab")
       (effects (font (size 1 1) (thickness 0.15)))
@@
     (property "Sheetfile" "ioBoard.kicad_sch")
     (property "Sheetname" "")
-    (attr exclude_from_pos_files)
+    (attr exclude_from_pos_files exclude_from_bom)
     (fp_text reference "H1" (at 0 -3.2) (layer "F.Fab")
       (effects (font (size 1 1) (thickness 0.15)))
@@
     (property "Sheetfile" "ioBoard.kicad_sch")
     (property "Sheetname" "")
-    (attr smd)
+    (attr smd exclude_from_pos_files exclude_from_bom)
     (fp_text reference "J2" (at 0 -7.0104 unlocked) (layer "F.Fab")
       (effects (font (size 1 1) (thickness 0.15)))

Commit message: cleanup
Other:
- board text added: "IO-Board v1.0"
- board text removed: "IO-Board v.0.9"
Changed lines of the file:
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@@
   )
   (paper "A4")
+  (title_block
+    (title "IO-Board")
+    (date "2023-02-14")
+    (rev "1.0")
+    (company "Fabian Kuffer")
+  )
   (layers
     (0 "F.Cu" signal)
@@
   (gr_line (start 83.302 121.92) (end 111.698 121.92) (layer "Edge.Cuts") (width 0.1))
   (gr_line (start 97.5 124.46) (end 97.5 94.488) (layer "User.1") (width 0.15))
-  (gr_text "IO-Board\nv.0.9" (at 97.536 93.98) (layer "B.SilkS")
+  (gr_text "IO-Board\nv1.0" (at 97.536 93.98) (layer "B.SilkS")
     (effects (font (size 1 1) (thickness 0.15)) (justify mirror))
   )
