File: ioBoard/ioBoard.kicad_sch (KiCad schematic)
At the start: 23 parts, among them J1 Conn_01x06_Male, J2 Conn_01x14, SW1 SW_Push, SW2 SW_Push

Commit message: io board pcb created
Parts:
- C1, C2: value 105u -> 1u; footprint (none) -> Capacitor_SMD:C_0805_2012Metric_Pad1.18x1.45mm_HandSolder
- C3, C4, C5, C6, C7, C8: footprint (none) -> Capacitor_SMD:C_0402_1005Metric_Pad0.74x0.62mm_HandSolder
- D1: footprint (none) -> Diode_SMD:D_SMA
- H1, H2, H3, H4: footprint (none) -> MountingHole:MountingHole_2.2mm_M2
- J1: footprint (none) -> Connector_JST:JST_GH_SM06B-GHS-TB_1x06-1MP_P1.25mm_Horizontal
- J2: footprint (none) -> SSD1306:SSD1306_Display_14PIN
- R1, R2, R3, R4, R5, R6: footprint (none) -> Resistor_SMD:R_0402_1005Metric
- SW1, SW2: value SW_Push -> C202424; footprint (none) -> Button_Switch_SMD:SW_SPST_SKQG_WithStem
